File: TP_DCI.sch (KiCad schematic (older format))
At the start: 32 parts, among them J1 Conn_01x02_Male, J2 Conn_01x07_Female, J3 Conn_01x07_Female, SW1 SW_DIP_x03, U1 MAX3157CAI+, U2 TPS54232

Commit message: Avanzo con esquematico
Parts:
- removed J1: Conn_01x02_Male, symbol Connector:Conn_01x02_Male
- removed J2, J3: Conn_01x07_Female, symbol Connector:Conn_01x07_Female
- removed J?: Conn_01x06_Male, symbol Connector:Conn_01x06_Male
- added J? (x2): Conn_01x14_Female, symbol Connector:Conn_01x14_Female
- added X1: Screw_Terminal_01x06, symbol Connector:Screw_Terminal_01x06
- added X2: Screw_Terminal_01x02, symbol Connector:Screw_Terminal_01x02
Connections:
- net labels added: 6, 7, A5, A6, RX, TX, U2_FB, VS
- wire segments 32 -> 59
- no-connect marks 0 -> 19
Other:
- note added: "Fuente de Alimentacion:"
- note added: "Integrado principal:"
- moved on the sheet: C1, C10, C11, C2, C3, C4, C5, C6, C7, C8, C9, D1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

Commit message: Avanzo con asociacion de footprints
Parts:
- added JP1, JP2, JP3, JP4: SolderJumper_2_Open, Jumper:SolderJumper-2_P1.3mm_Open_RoundedPad1.0x1.5mm, symbol Jumper:SolderJumper_2_Open
- D1: footprint (none) -> DO_214AC:DO-214AC
- FID1: footprint (none) -> Fiducial:Fiducial_0.5mm_Mask1.5mm
- J1, J2: renamed from J?; footprint (none) -> Connector_PinSocket_1.27mm:PinSocket_1x14_P1.27mm_Vertical
- R7, R8: value DNP -> DNP*
- SW1: footprint (none) -> Button_Switch_THT:SW_DIP_SPSTx03_Slide_6.7x9.18mm_W7.62mm_P2.54mm_LowProfile
- U1: footprint SOP65P777X199-28N -> MAX3157:SOP65P777X199-28N
- X1: footprint (none) -> TerminalBlock_Phoenix:TerminalBlock_Phoenix_MKDS-1,5-6-5.08_1x06_P5.08mm_Horizontal
- X2: footprint (none) -> TerminalBlock_Phoenix:TerminalBlock_Phoenix_MKDS-1,5-2-5.08_1x02_P5.08mm_Horizontal
Connections:
- net 6: now also JP4.1 (A); no longer U1.27 (RXP)
- net 7: now also JP3.1 (A); no longer U1.26 (TXP)
- net A5: now also JP1.1 (A); no longer R7.1, U1.2 (#RE)
- net A6: now also JP2.1 (A)
- net GND: now also R8.2, U2.7 (GND); no longer R8.1
- net TX: now also J2.6 (Pin_6)
- net A6_jmp: now reaches U1.3 (DE)
- net A6_jmp: now also R8.1, JP2.2 (B); no longer R8.2
- new net 6_jmp: JP4.2 (B), U1.27 (RXP)
- new net 7_jmp: JP3.2 (B), U1.26 (TXP)
- new net A5_jmp: JP1.2 (B), R7.1, U1.2 (#RE)
Other:
- note added: "*DNP: Do Not Populate"
- moved on the sheet: C10, C11, C6, C7, C8, C9, D1, FID1, J1, J2, L1, R1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

Commit message: Fin etapa 1, esquematico y asociacion de footprints
Parts:
- removed J1, J2: Conn_01x14_Female, Connector_PinSocket_1.27mm:PinSocket_1x14_P1.27mm_Vertical, symbol Connector:Conn_01x14_Female
- added ShieldMKR1: _WIFI_1010, MKR:MKR_WIFI_1010_Shield, symbol MKR:_WIFI_1010
- C1, C2, C4, C5, C6, C7: footprint (none) -> Capacitor_SMD:C_0805_2012Metric
- C10, C8: footprint (none) -> Capacitor_THT:C_Disc_D3.0mm_W1.6mm_P2.50mm
- C11, C9: footprint (none) -> Capacitor_THT:CP_Radial_D4.0mm_P1.50mm
- C3: footprint (none) -> Capacitor_Tantalum_SMD:CP_EIA-1608-08_AVX-J
- D1: value D_Schottky -> SS24FL; footprint DO_214AC:DO-214AC -> DO_214AC:DO-214BA
- L1: footprint (none) -> L_15uh:IND_#A921CY-150M=P3
- R1, R10, R11, R2, R3, R4, R5, R6, R7, R8, R9: footprint (none) -> Resistor_SMD:R_0805_2012Metric
Connections:
- net +3V3: now also ShieldMKR1.26 (+3V3)
- net +5V: now also ShieldMKR1.28 (+5V)
- net 6: now also ShieldMKR1.15 (D6)
- net 7: now also ShieldMKR1.16 (D7)
- net A5: now also ShieldMKR1.7 (A5)
- net A6: now also ShieldMKR1.8 (A6)
- net GND: now also ShieldMKR1.25 (GND)
- net RX: now also ShieldMKR1.22 (D13/RX)
- net TX: now also ShieldMKR1.23 (D14/TX)
- net VS: now also ShieldMKR1.27 (VIN)

Commit message: Para correccion Etapa 1
Connections:
- net GND: no longer R2.1
- net H_#F: now also R11.1, SW1.2; no longer R2.2, SW1.3
- net ISOGND: now also C2.2, U1.14 (IGND)
- net ISOVCC: now also R11.2
- net Y: now also R2.1; no longer R11.2
- new net: R2.2, SW1.3
Other:
- moved on the sheet: C2, R2
Changed lines of the file:
@@
-$EndComp
-$Comp
-L Device:R R2
-U 1 1 605D77BB
-P 8450 3900
-F 0 "R2" V 8657 3900 50  0000 C CNN
-F 1 "120" V 8566 3900 50  0000 C CNN
-F 2 "Resistor_SMD:R_0805_2012Metric" V 8380 3900 50  0001 C CNN
-F 3 "~" H 8450 3900 50  0001 C CNN
-	1    8450 3900
-	0    -1   -1   0
 $EndComp
 $Comp
@@
 L Device:C C2
 U 1 1 605DCB3D
-P 7150 2200
-F 0 "C2" V 6898 2200 50  0000 C CNN
-F 1 "10n" V 6989 2200 50  0000 C CNN
-F 2 "Capacitor_SMD:C_0805_2012Metric" H 7188 2050 50  0001 C CNN
-F 3 "~" H 7150 2200 50  0001 C CNN
-	1    7150 2200
-	0    1    1    0
+P 7000 2350
+F 0 "C2" V 6748 2350 50  0000 C CNN
+F 1 "10n" V 6839 2350 50  0000 C CNN
+F 2 "Capacitor_SMD:C_0805_2012Metric" H 7038 2200 50  0001 C CNN
+F 3 "~" H 7000 2350 50  0001 C CNN
+	1    7000 2350
+	-1   0    0    1
 $EndComp
 $Comp
@@
 L power:GND #PWR0102
 U 1 1 606F44E7
-P 7350 2200
-F 0 "#PWR0102" H 7350 1950 50  0001 C CNN
-F 1 "GND" H 7355 2027 50  0000 C CNN
-F 2 "" H 7350 2200 50  0001 C CNN
-F 3 "" H 7350 2200 50  0001 C CNN
-	1    7350 2200
-	1    0    0    -1
-$EndComp
-Wire Wire Line
-	7300 2200 7350 2200
+P 7000 2550
+F 0 "#PWR0102" H 7000 2300 50  0001 C CNN
+F 1 "GND" H 7005 2377 50  0000 C CNN
+F 2 "" H 7000 2550 50  0001 C CNN
+F 3 "" H 7000 2550 50  0001 C CNN
+	1    7000 2550
+	1    0    0    -1
+$EndComp
 Wire Wire Line
 	9550 3700 9500 3700
 Wire Wire Line
-	9000 3800 9550 3800
-Wire Wire Line
-	8600 3900 9100 3900
-Wire Wire Line
-	9100 3900 9100 4000
-Connection ~ 9100 3900
-Wire Wire Line
-	9100 3900 9550 3900
-$Comp
-L power:GND #PWR0103
-U 1 1 6075513E
-P 8150 3900
-F 0 "#PWR0103" H 8150 3650 50  0001 C CNN
-F 1 "GND" H 8155 3727 50  0000 C CNN
-F 2 "" H 8150 3900 50  0001 C CNN
-F 3 "" H 8150 3900 50  0001 C CNN
-	1    8150 3900
-	1    0    0    -1
-$EndComp
-Wire Wire Line
-	8300 3900 8150 3900
+	9000 3800 9100 3800
 Wire Wire Line
 	6300 1400 6400 1400
@@
 Text Label 10150 3900 0    50   ~ 0
 Z
-Text Label 8700 3800 2    50   ~ 0
+Text Label 8100 3900 2    50   ~ 0
 Y
 Text Label 5600 5650 0    50   ~ 0
@@
 Text Label 2000 2350 0    50   ~ 0
 7
+Wire Wire Line
+	9100 4000 9100 3800
+Connection ~ 9100 3800
+Wire Wire Line
+	9100 3800 9550 3800
+Text Label 8700 3800 2    50   ~ 0
+ISOVCC
+Wire Wire Line
+	8400 3900 9550 3900
+$Comp
+L Device:R R2
+U 1 1 605D77BB
+P 8250 3900
+F 0 "R2" V 8457 3900 50  0000 C CNN
+F 1 "120" V 8366 3900 50  0000 C CNN
+F 2 "Resistor_SMD:R_0805_2012Metric" V 8180 3900 50  0001 C CNN
+F 3 "~" H 8250 3900 50  0001 C CNN
+	1    8250 3900
+	0    -1   -1   0
+$EndComp
+Wire Wire Line
+	7000 2550 7000 2500
+Text Label 7100 2200 0    50   ~ 0
+ISOGND
+Wire Wire Line
+	7000 2200 7100 2200
+Connection ~ 7000 2200
 $EndSCHEMATC

Commit message: Agrego correcciones de Gaspar
Parts:
- added FID2, FID3, FID4: Fiducial, Fiducial:Fiducial_0.5mm_Mask1.5mm, symbol Mechanical:Fiducial
- Interconexion1: renamed from ShieldMKR1; value _WIFI_1010 -> MKR1_WIFI_1010
Other:
- note added: "Bornera de conexion:"
- note added: "Conexion con placa MKR1_Wifi1010:"
- note added: "Jumpers:"
- note added: "Selectora:"
- moved on the sheet: C1, C10, C11, C2, C3, C4, C5, C6, C7, C8, C9, D1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

Commit message: Lista para correccion
Other:
- note added: "Creative Commons Attribution-ShareAlike 4.0 International License"
Changed lines of the file:
@@
 Text Notes 5350 3700 0    50   ~ 0
 Bornera de conexion:
+Text Notes 600  7700 0    50   Italic 0
+Creative Commons Attribution-ShareAlike 4.0 International License
 $EndSCHEMATC
