File: TP_DCI.sch (KiCad schematic (older format))
At the start: 38 parts, among them SW1 SW_DIP_x03, U1 MAX3157CAI+, U2 TPS54232, X1 Screw_Terminal_01x06, X2 Screw_Terminal_01x02

Commit message: Arranco con el PCB
Parts:
- C10, C8: footprint Capacitor_THT:C_Disc_D3.0mm_W1.6mm_P2.50mm -> Capacitor_Tantalum_SMD:CP_EIA-1608-08_AVX-J
- C11, C9: footprint Capacitor_THT:CP_Radial_D4.0mm_P1.50mm -> Capacitor_Tantalum_SMD:CP_EIA-1608-08_AVX-J
Connections:
- net A: now also X1.5 (Pin_5); no longer X1.2 (Pin_2)
- net B: now also X1.4 (Pin_4); no longer X1.3 (Pin_3)
- net ISOGND: now also X1.6 (Pin_6); no longer X1.1 (Pin_1)
- net ISOVCC: now also X1.1 (Pin_1); no longer X1.6 (Pin_6)
- net Y: now also X1.3 (Pin_3); no longer X1.4 (Pin_4)
- net Z: now also X1.2 (Pin_2); no longer X1.5 (Pin_5)
Changed lines of the file:
@@
 F 0 "C10" V 4752 5650 50  0000 C CNN
 F 1 "100n" V 4661 5650 50  0000 C CNN
-F 2 "Capacitor_THT:C_Disc_D3.0mm_W1.6mm_P2.50mm" H 4538 5500 50  0001 C CNN
+F 2 "Capacitor_Tantalum_SMD:CP_EIA-1608-08_AVX-J" H 4538 5500 50  0001 C CNN
 F 3 "~" H 4500 5650 50  0001 C CNN
 	1    4500 5650
@@
 F 0 "C11" H 6165 5846 50  0000 L CNN
 F 1 "10u" H 6165 5755 50  0000 L CNN
-F 2 "Capacitor_THT:CP_Radial_D4.0mm_P1.50mm" H 6088 5650 50  0001 C CNN
+F 2 "Capacitor_Tantalum_SMD:CP_EIA-1608-08_AVX-J" H 6088 5650 50  0001 C CNN
 F 3 "~" H 6050 5800 50  0001 C CNN
 	1    6050 5800
@@
 F 0 "C8" H 2365 6346 50  0000 L CNN
 F 1 "110p" H 2365 6255 50  0000 L CNN
-F 2 "Capacitor_THT:C_Disc_D3.0mm_W1.6mm_P2.50mm" H 2288 6150 50  0001 C CNN
+F 2 "Capacitor_Tantalum_SMD:CP_EIA-1608-08_AVX-J" H 2288 6150 50  0001 C CNN
 F 3 "~" H 2250 6300 50  0001 C CNN
 	1    2250 6300
@@
 F 0 "C9" H 2065 5946 50  0000 L CNN
 F 1 "10u" H 2065 5855 50  0000 L CNN
-F 2 "Capacitor_THT:CP_Radial_D4.0mm_P1.50mm" H 1988 5750 50  0001 C CNN
+F 2 "Capacitor_Tantalum_SMD:CP_EIA-1608-08_AVX-J" H 1988 5750 50  0001 C CNN
 F 3 "~" H 1950 5900 50  0001 C CNN
 	1    1950 5900
@@
 Text Label 6450 2700 0    50   ~ 0
 ISOGND
+Text Label 5500 4400 2    50   ~ 0
+ISOGND
+Text Label 5500 4300 2    50   ~ 0
+A
+Text Label 5500 4200 2    50   ~ 0
+B
+Text Label 5500 4100 2    50   ~ 0
+Y
+Text Label 5500 4000 2    50   ~ 0
+Z
 Text Label 5500 3900 2    50   ~ 0
-ISOGND
-Text Label 5500 4000 2    50   ~ 0
-A
-Text Label 5500 4100 2    50   ~ 0
-B
-Text Label 5500 4200 2    50   ~ 0
-Y
-Text Label 5500 4300 2    50   ~ 0
-Z
-Text Label 5500 4400 2    50   ~ 0
 ISOVCC
 Text Label 9150 4100 2    50   ~ 0
@@
 L power:PWR_FLAG #FLG0104
 U 1 1 607D8A39
-P 5100 4400
-F 0 "#FLG0104" H 5100 4475 50  0001 C CNN
-F 1 "PWR_FLAG" H 5100 4573 50  0000 C CNN
-F 2 "" H 5100 4400 50  0001 C CNN
-F 3 "~" H 5100 4400 50  0001 C CNN
-	1    5100 4400
-	1    0    0    -1
-$EndComp
-Wire Wire Line
-	5100 4400 5500 4400
+P 5100 3900
+F 0 "#FLG0104" H 5100 3975 50  0001 C CNN
+F 1 "PWR_FLAG" H 5100 4073 50  0000 C CNN
+F 2 "" H 5100 3900 50  0001 C CNN
+F 3 "~" H 5100 3900 50  0001 C CNN
+	1    5100 3900
+	1    0    0    -1
+$EndComp
+Wire Wire Line
+	5100 3900 5500 3900
 $Comp
 L power:PWR_FLAG #FLG0105
@@
 Text Notes 9600 3650 0    50   ~ 0
 Selectora:
-Text Notes 5350 3700 0    50   ~ 0
+Text Notes 5550 3750 0    50   ~ 0
 Bornera de conexion:
 Text Notes 600  7700 0    50   Italic 0

Commit message: Version del PCB completa
Parts:
- added H1, H2, H3, H4: MountingHole, MountingHole:MountingHole_2.1mm, symbol Mechanical:MountingHole
- C11, C3, C9: footprint Capacitor_Tantalum_SMD:CP_EIA-1608-08_AVX-J -> Capacitor_SMD:C_0805_2012Metric
Connections:
- net A: now also SW1.2, X1.4 (Pin_4); no longer SW1.6, X1.5 (Pin_5)
- net B: now also R1.2, X1.5 (Pin_5); no longer R1.1, X1.4 (Pin_4)
- net GND: now also X2.2 (Pin_2); no longer X2.1 (Pin_1)
- net H_#F: now also SW1.1; no longer SW1.2
- net ISOGND: now also SW1.6, X1.2 (Pin_2); no longer SW1.5, X1.6 (Pin_6)
- net Y: now also X1.6 (Pin_6); no longer X1.3 (Pin_3)
- net Z: now also X1.3 (Pin_3); no longer X1.2 (Pin_2)
- net at C9.1, U2.2 (VIN): now also X2.1 (Pin_1); no longer X2.2 (Pin_2)
- new net: R1.1, SW1.5
Other:
- moved on the sheet: R1, R11, R2, SW1
Changed lines of the file:
@@
 L Switch:SW_DIP_x03 SW1
 U 1 1 605D3E29
-P 9800 4300
-F 0 "SW1" H 9800 4767 50  0000 C CNN
-F 1 "SW_DIP_x03" H 9800 4676 50  0000 C CNN
-F 2 "Button_Switch_THT:SW_DIP_SPSTx03_Slide_6.7x9.18mm_W7.62mm_P2.54mm_LowProfile" H 9800 4300 50  0001 C CNN
-F 3 "~" H 9800 4300 50  0001 C CNN
-	1    9800 4300
+P 9350 4400
+F 0 "SW1" H 9350 4867 50  0000 C CNN
+F 1 "SW_DIP_x03" H 9350 4776 50  0000 C CNN
+F 2 "Button_Switch_THT:SW_DIP_SPSTx03_Slide_6.7x9.18mm_W7.62mm_P2.54mm_LowProfile" H 9350 4400 50  0001 C CNN
+F 3 "~" H 9350 4400 50  0001 C CNN
+	1    9350 4400
 	1    0    0    -1
 $EndComp
@@
 	1    2750 6200
 	1    0    0    -1
-$EndComp
-$Comp
-L Device:R R1
-U 1 1 605D7B9F
-P 9300 4100
-F 0 "R1" V 9507 4100 50  0000 C CNN
-F 1 "120" V 9416 4100 50  0000 C CNN
-F 2 "Resistor_SMD:R_0805_2012Metric" V 9230 4100 50  0001 C CNN
-F 3 "~" H 9300 4100 50  0001 C CNN
-	1    9300 4100
-	0    -1   -1   0
 $EndComp
 $Comp
@@
 F 0 "C3" V 7552 1400 50  0000 C CNN
 F 1 "1u" V 7461 1400 50  0000 C CNN
-F 2 "Capacitor_Tantalum_SMD:CP_EIA-1608-08_AVX-J" H 7338 1250 50  0001 C CNN
+F 2 "Capacitor_SMD:C_0805_2012Metric" H 7338 1250 50  0001 C CNN
 F 3 "~" H 7300 1400 50  0001 C CNN
 	1    7300 1400
@@
 F 0 "C11" H 6165 5846 50  0000 L CNN
 F 1 "10u" H 6165 5755 50  0000 L CNN
-F 2 "Capacitor_Tantalum_SMD:CP_EIA-1608-08_AVX-J" H 6088 5650 50  0001 C CNN
+F 2 "Capacitor_SMD:C_0805_2012Metric" H 6088 5650 50  0001 C CNN
 F 3 "~" H 6050 5800 50  0001 C CNN
 	1    6050 5800
@@
 L Device:R R11
 U 1 1 605FBEDB
-P 8800 4200
-F 0 "R11" V 8593 4200 50  0000 C CNN
-F 1 "10k2" V 8684 4200 50  0000 C CNN
-F 2 "Resistor_SMD:R_0805_2012Metric" V 8730 4200 50  0001 C CNN
-F 3 "~" H 8800 4200 50  0001 C CNN
-	1    8800 4200
+P 8675 4200
+F 0 "R11" V 8468 4200 50  0000 C CNN
+F 1 "10k2" V 8559 4200 50  0000 C CNN
+F 2 "Resistor_SMD:R_0805_2012Metric" V 8605 4200 50  0001 C CNN
+F 3 "~" H 8675 4200 50  0001 C CNN
+	1    8675 4200
 	0    1    1    0
 $EndComp
@@
 F 0 "C9" H 2065 5946 50  0000 L CNN
 F 1 "10u" H 2065 5855 50  0000 L CNN
-F 2 "Capacitor_Tantalum_SMD:CP_EIA-1608-08_AVX-J" H 1988 5750 50  0001 C CNN
+F 2 "Capacitor_SMD:C_0805_2012Metric" H 1988 5750 50  0001 C CNN
 F 3 "~" H 1950 5900 50  0001 C CNN
 	1    1950 5900
@@
 $EndComp
 Wire Wire Line
-	9500 4100 9450 4100
-Wire Wire Line
-	8950 4200 9050 4200
-Wire Wire Line
 	6450 1500 6550 1500
 Wire Wire Line
@@
 Wire Wire Line
 	1950 5650 1950 5750
-Wire Wire Line
-	1400 5650 1950 5650
 Connection ~ 1950 5650
 $Comp
@@
 L Connector:Screw_Terminal_01x02 X2
 U 1 1 607D2105
-P 1200 5750
-F 0 "X2" H 1150 5400 50  0000 L CNN
-F 1 "Screw_Terminal_01x02" H 750 5500 50  0000 L CNN
-F 2 "TerminalBlock_Phoenix:TerminalBlock_Phoenix_MKDS-1,5-2-5.08_1x02_P5.08mm_Horizontal" H 1200 5750 50  0001 C CNN
-F 3 "~" H 1200 5750 50  0001 C CNN
-	1    1200 5750
-	-1   0    0    1
+P 1200 5650
+F 0 "X2" H 1300 5600 50  0000 L CNN
+F 1 "Screw_Terminal_01x02" H 900 5800 50  0000 L CNN
+F 2 "TerminalBlock_Phoenix:TerminalBlock_Phoenix_MKDS-1,5-2-5.08_1x02_P5.08mm_Horizontal" H 1200 5650 50  0001 C CNN
+F 3 "~" H 1200 5650 50  0001 C CNN
+	1    1200 5650
+	-1   0    0    -1
 $EndComp
 $Comp
@@
 Text Label 6450 2700 0    50   ~ 0
 ISOGND
+Text Label 5500 4000 2    50   ~ 0
+ISOGND
+Text Label 5500 4200 2    50   ~ 0
+A
+Text Label 5500 4300 2    50   ~ 0
+B
 Text Label 5500 4400 2    50   ~ 0
-ISOGND
-Text Label 5500 4300 2    50   ~ 0
-A
-Text Label 5500 4200 2    50   ~ 0
-B
+Y
 Text Label 5500 4100 2    50   ~ 0
-Y
-Text Label 5500 4000 2    50   ~ 0
 Z
 Text Label 5500 3900 2    50   ~ 0
 ISOVCC
-Text Label 9150 4100 2    50   ~ 0
+Text Label 10400 4300 0    50   ~ 0
 B
-Text Label 9050 4500 2    50   ~ 0
+Text Label 8825 4350 2    50   ~ 0
 H_#F
-Text Label 10100 4100 0    50   ~ 0
+Text Label 9050 4300 2    50   ~ 0
 A
-Text Label 10100 4200 0    50   ~ 0
+Text Label 9650 4200 0    50   ~ 0
 ISOGND
-Text Label 10100 4300 0    50   ~ 0
+Text Label 9650 4400 0    50   ~ 0
 Z
-Text Label 8050 4300 2    50   ~ 0
+Text Label 7950 4400 2    50   ~ 0
 Y
 Text Label 5550 6050 0    50   ~ 0
@@
 Text Label 2100 2700 0    50   ~ 0
 7
-Wire Wire Line
-	9050 4500 9050 4200
-Connection ~ 9050 4200
-Wire Wire Line
-	9050 4200 9500 4200
-Text Label 8650 4200 2    50   ~ 0
+Text Label 8525 4200 2    50   ~ 0
 ISOVCC
-Wire Wire Line
-	8350 4300 9500 4300
 $Comp
 L Device:R R2
 U 1 1 605D77BB
-P 8200 4300
-F 0 "R2" V 8407 4300 50  0000 C CNN
-F 1 "120" V 8316 4300 50  0000 C CNN
-F 2 "Resistor_SMD:R_0805_2012Metric" V 8130 4300 50  0001 C CNN
-F 3 "~" H 8200 4300 50  0001 C CNN
-	1    8200 4300
+P 8100 4400
+F 0 "R2" V 8307 4400 50  0000 C CNN
+F 1 "120" V 8216 4400 50  0000 C CNN
+F 2 "Resistor_SMD:R_0805_2012Metric" V 8030 4400 50  0001 C CNN
+F 3 "~" H 8100 4400 50  0001 C CNN
+	1    8100 4400
 	0    -1   -1   0
 $EndComp
@@
 $EndComp
 Wire Wire Line
-	1400 5750 1500 5750
-Wire Wire Line
 	1950 5650 3450 5650
 Connection ~ 6050 5650
@@
 Text Notes 1650 3700 0    50   ~ 0
 Jumpers:
-Text Notes 9600 3650 0    50   ~ 0
+Text Notes 9150 3750 0    50   ~ 0
 Selectora:
 Text Notes 5550 3750 0    50   ~ 0
@@
 Text Notes 600  7700 0    50   Italic 0
 Creative Commons Attribution-ShareAlike 4.0 International License
+Wire Wire Line
+	1400 5750 1500 5750
+Wire Wire Line
+	1400 5650 1950 5650
+Wire Wire Line
+	8825 4350 8825 4200
+Connection ~ 8825 4200
+Wire Wire Line
+	8825 4200 9050 4200
+Wire Wire Line
+	10300 4300 10400 4300
+Wire Wire Line
+	9650 4300 10000 4300
+$Comp
+L Device:R R1
+U 1 1 605D7B9F
+P 10150 4300
+F 0 "R1" V 10357 4300 50  0000 C CNN
+F 1 "120" V 10266 4300 50  0000 C CNN
+F 2 "Resistor_SMD:R_0805_2012Metric" V 10080 4300 50  0001 C CNN
+F 3 "~" H 10150 4300 50  0001 C CNN
+	1    10150 4300
+	0    -1   -1   0
+$EndComp
+Wire Wire Line
+	8250 4400 9050 4400
+$Comp
+L Mechanical:MountingHole H1
+U 1 1 6084B85C
+P 9750 750
+F 0 "H1" H 9850 796 50  0000 L CNN
+F 1 "MountingHole" H 9850 705 50  0000 L CNN
+F 2 "MountingHole:MountingHole_2.1mm" H 9750 750 50  0001 C CNN
+F 3 "~" H 9750 750 50  0001 C CNN
+	1    9750 750
+	1    0    0    -1
+$EndComp
+$Comp
+L Mechanical:MountingHole H2
+U 1 1 6084C43C
+P 9750 1000
+F 0 "H2" H 9850 1046 50  0000 L CNN
+F 1 "MountingHole" H 9850 955 50  0000 L CNN
+F 2 "MountingHole:MountingHole_2.1mm" H 9750 1000 50  0001 C CNN
+F 3 "~" H 9750 1000 50  0001 C CNN
+	1    9750 1000
+	1    0    0    -1
+$EndComp
+$Comp
+L Mechanical:MountingHole H3
+U 1 1 6084CC49
+P 9750 1250
+F 0 "H3" H 9850 1296 50  0000 L CNN
+F 1 "MountingHole" H 9850 1205 50  0000 L CNN
+F 2 "MountingHole:MountingHole_2.1mm" H 9750 1250 50  0001 C CNN
+F 3 "~" H 9750 1250 50  0001 C CNN
+	1    9750 1250
+	1    0    0    -1
+$EndComp
+$Comp
+L Mechanical:MountingHole H4
+U 1 1 6084D8AE
+P 9750 1500
+F 0 "H4" H 9850 1546 50  0000 L CNN
+F 1 "MountingHole" H 9850 1455 50  0000 L CNN
+F 2 "MountingHole:MountingHole_2.1mm" H 9750 1500 50  0001 C CNN
+F 3 "~" H 9750 1500 50  0001 C CNN
+	1    9750 1500
+	1    0    0    -1
+$EndComp
 $EndSCHEMATC

Commit message: Version para corregir PCB
Parts:
- D1: Mouser (none) -> 512-SS24FL
- L1: Mouser (none) -> 710-7447707150
- SW1: Mouser (none) -> 490-DS01C-254-S-03BE
- U1: Mouser (none) -> 700-MAX3157CAI+
- U2: Mouser (none) -> 595-TPS54232D
- XA1: renamed from Interconexion1; RAM size 32KBytes -> (none); automotive No -> (none); category UNK -> (none); core architecture ARM Cortex-M0+ -> (none); data bus width 32bits -> (none); device class L1 Integrated Circuits (ICs) -> (none); device class L2 Embedded Processors and Controllers -> (none); device class L3 Microcontrollers -> (none); digikey description ARDUINO MKR WIFI 1010 -> (none); digikey part number 1050-1162-ND -> (none); frequency 48MHz -> (none); interface I2C,SPI,UART,I2S -> (none); lead free Yes -> (none); library id 7eb282d1527b7afb -> (none); manufacturer Arduino -> (none); max supply voltage 5V -> (none); memory size 256KBytes -> (none); memory type FLASH -> (none); min supply voltage 3.3V -> (none); mouser part number 782-ABX00023 -> (none); number of A/D converters 1 -> (none); number of ADC channels 7 -> (none); number of I/Os 8 -> (none); number of I2C channels 1 -> (none); number of PWM channels 12 -> (none); number of SPI channels 1 -> (none); number of UART channels 1 -> (none); package EVALUATION_BOARD -> (none); rohs Yes -> (none)
Connections:
- net U2_FB: no longer names the net of R10.1, R9.2, U2.5 (FB)
Other:
- moved on the sheet: C11, C2
