File: TP_DCI.sch (KiCad schematic (older format))
At the start: 42 parts, among them SW1 SW_DIP_x03, U1 MAX3157CAI+, U2 TPS54232, X1 Screw_Terminal_01x06, X2 Screw_Terminal_01x02

Commit message: Agrego correcciones
Parts:
- removed FID3, FID4: Fiducial, Fiducial:Fiducial_0.5mm_Mask1.5mm, symbol Mechanical:Fiducial
Changed lines of the file:
@@
-	1    0    0    -1
-$EndComp
-$Comp
-L Mechanical:Fiducial FID3
-U 1 1 6098FB8D
-P 10700 1250
-F 0 "FID3" H 10785 1296 50  0000 L CNN
-F 1 "Fiducial" H 10785 1205 50  0000 L CNN
-F 2 "Fiducial:Fiducial_0.5mm_Mask1.5mm" H 10700 1250 50  0001 C CNN
-F 3 "~" H 10700 1250 50  0001 C CNN
-	1    10700 1250
-	1    0    0    -1
-$EndComp
-$Comp
-L Mechanical:Fiducial FID4
-U 1 1 60991997
-P 10700 1500
-F 0 "FID4" H 10785 1546 50  0000 L CNN
-F 1 "Fiducial" H 10785 1455 50  0000 L CNN
-F 2 "Fiducial:Fiducial_0.5mm_Mask1.5mm" H 10700 1500 50  0001 C CNN
-F 3 "~" H 10700 1500 50  0001 C CNN
-	1    10700 1500
 	1    0    0    -1
 $EndComp
@@
 	1    0    0    -1
 $EndComp
-$Comp
-L Mechanical:MountingHole H3
-U 1 1 6084CC49
-P 9750 1250
-F 0 "H3" H 9850 1296 50  0000 L CNN
-F 1 "MountingHole" H 9850 1205 50  0000 L CNN
-F 2 "MountingHole:MountingHole_2.1mm" H 9750 1250 50  0001 C CNN
-F 3 "~" H 9750 1250 50  0001 C CNN
-	1    9750 1250
-	1    0    0    -1
-$EndComp
-$Comp
-L Mechanical:MountingHole H4
-U 1 1 6084D8AE
-P 9750 1500
-F 0 "H4" H 9850 1546 50  0000 L CNN
-F 1 "MountingHole" H 9850 1455 50  0000 L CNN
-F 2 "MountingHole:MountingHole_2.1mm" H 9750 1500 50  0001 C CNN
-F 3 "~" H 9750 1500 50  0001 C CNN
-	1    9750 1500
-	1    0    0    -1
-$EndComp
 Wire Wire Line
 	1100 4100 1150 4100
@@
 Wire Wire Line
 	5450 6050 5450 6150
+$Comp
+L Mechanical:MountingHole H3
+U 1 1 608CC8EF
+P 9750 1225
+F 0 "H3" H 9850 1271 50  0000 L CNN
+F 1 "MountingHole" H 9850 1180 50  0000 L CNN
+F 2 "MountingHole:MountingHole_2.1mm" H 9750 1225 50  0001 C CNN
+F 3 "~" H 9750 1225 50  0001 C CNN
+	1    9750 1225
+	1    0    0    -1
+$EndComp
+$Comp
+L Mechanical:MountingHole H4
+U 1 1 608CC8F5
+P 9750 1475
+F 0 "H4" H 9850 1521 50  0000 L CNN
+F 1 "MountingHole" H 9850 1430 50  0000 L CNN
+F 2 "MountingHole:MountingHole_2.1mm" H 9750 1475 50  0001 C CNN
+F 3 "~" H 9750 1475 50  0001 C CNN
+	1    9750 1475
+	1    0    0    -1
+$EndComp
 $EndSCHEMATC

Commit message: Agrego correcciones finales
Parts:
- X2: footprint TerminalBlock_Phoenix:TerminalBlock_Phoenix_MKDS-1,5-2-5.08_1x02_P5.08mm_Horizontal -> TerminalBlock:TerminalBlock_bornier-2_P5.08mm
Changed lines of the file:
@@
 F 0 "X2" H 1300 5600 50  0000 L CNN
 F 1 "Screw_Terminal_01x02" H 900 5800 50  0000 L CNN
-F 2 "TerminalBlock_Phoenix:TerminalBlock_Phoenix_MKDS-1,5-2-5.08_1x02_P5.08mm_Horizontal" H 1200 5650 50  0001 C CNN
+F 2 "TerminalBlock:TerminalBlock_bornier-2_P5.08mm" H 1200 5650 50  0001 C CNN
 F 3 "~" H 1200 5650 50  0001 C CNN
 	1    1200 5650
