File: TP_DCI.kicad_pcb (KiCad board)
At the start: 2 copper layers, 35 parts, among them SW1 SW_DIP_x03, U1 MAX3157CAI+, U2 TPS54232, X1 Screw_Terminal_01x06, X2 Screw_Terminal_01x02

Commit message: Para correccion Etapa 1
Parts:
- moved C3 15.3 mm to (152.7, 100.1)
- moved C7 15.3 mm to (137.5, 115.5)
- moved FID1 15.3 mm to (141.2, 115.6)
- moved JP1 15.3 mm to (170.0, 99.2)
- moved JP3 15.3 mm to (174.4, 95.5)
- moved R1 15.3 mm to (165.6, 96.0)
- moved R10 15.3 mm to (165.6, 98.9)
- moved R11 15.3 mm to (173.2, 89.3)
- moved R3 15.3 mm to (173.2, 92.3)
- moved R6 15.3 mm to (170.0, 96.0)
- moved SW1 15.3 mm to (160.0, 82.2)
- moved X2 15.3 mm to (149.7, 85.5)
- moved C2 15.3 mm to (133.0, 115.5)
- moved C4 15.3 mm to (128.6, 115.5)
- moved C5 15.3 mm to (124.1, 115.5)
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Connections:
- C2 pad 2: Net-(C2-Pad2) -> /ISOGND
- R11 pad 1: Net-(R11-Pad1) -> /H_#F
- R11 pad 2: /Y -> /ISOVCC
- R2 pad 1: GND -> /Y
- R2 pad 2: /H_#F -> Net-(R2-Pad2)
- SW1 pad 2: Net-(R11-Pad1) -> /H_#F
- SW1 pad 3: /H_#F -> Net-(R2-Pad2)
- U1 pad 14: Net-(C2-Pad2) -> /ISOGND

Commit message: Agrego correcciones de Gaspar
Parts:
- added FID2: Fiducial, Fiducial:Fiducial_0.5mm_Mask1.5mm, F.Cu at (183.2, 76.3)
- added FID3: Fiducial, Fiducial:Fiducial_0.5mm_Mask1.5mm, F.Cu at (183.8, 84.8)
- added FID4: Fiducial, Fiducial:Fiducial_0.5mm_Mask1.5mm, F.Cu at (162.5, 109.0)
- moved C4 60.1 mm to (178.3, 81.8)
- moved C1 47.4 mm to (131.0, 111.0)
- moved C9 31.2 mm to (178.2, 77.5)
- moved R7 29.2 mm to (180.1, 87.8)
- moved C7 26.7 mm to (155.3, 95.7)
- moved JP2 26.7 mm to (181.3, 91.0)
- moved R8 23.4 mm to (163.2, 106.0)
- moved R2 22.9 mm to (172.5, 94.4)
- moved C5 20.7 mm to (144.3, 111.0)
- moved R1 18.3 mm to (180.1, 84.8)
- moved C6 16.8 mm to (135.4, 111.0)
- moved JP4 15.8 mm to (176.8, 94.7)
- moved R9 15.8 mm to (176.9, 91.4)
- moved C11 15.6 mm to (163.9, 95.8)
- moved R3 14.2 mm to (182.8, 81.8)
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Other:
- net class Default: clearance 0.2 -> 0.8; trace_width 0.25 -> 0.8
- rule trace_clearance: 0.2 -> 0.8
- board text added: "Fabricante MAYER: Ancho de pista: 0,8mm Vias: 1,6mm/0,8mm Margen global: 0,8mm"

Commit message: Arranco con el PCB
Parts:
- removed ShieldMKR1: _WIFI_1010, MKR:MKR_WIFI_1010_Shield
- added Interconexion1: MKR1_WIFI_1010, MKR:MKR_WIFI_1010_Shield, F.Cu at (117.0, 92.0)
- C10, C8: footprint Capacitor_THT:C_Disc_D3.0mm_W1.6mm_P2.50mm -> Capacitor_Tantalum_SMD:CP_EIA-1608-08_AVX-J
- C11, C9: footprint Capacitor_THT:CP_Radial_D4.0mm_P1.50mm -> Capacitor_Tantalum_SMD:CP_EIA-1608-08_AVX-J
- FID3, FID4: moved to B.Cu
- moved FID4 83.1 mm to (222.0, 51.0)
- moved C9 82.2 mm to (97.0, 90.5), turned to 90 degrees
- moved FID1 79.3 mm to (200.0, 51.0)
- moved X1 73.0 mm to (194.0, 103.0), turned to 90 degrees
- moved X2 69.1 mm to (88.0, 89.0), turned to 270 degrees
- moved R9 64.0 mm to (113.0, 96.0), turned to 270 degrees
- moved U2 62.0 mm to (104.0, 89.0)
- moved D1 59.1 mm to (115.0, 89.0), turned to 270 degrees
- moved R4 58.3 mm to (105.0, 95.9), turned to 270 degrees
- moved JP2 56.3 mm to (127.0, 106.0), turned to 270 degrees
- moved R10 55.7 mm to (117.0, 96.0), turned to 270 degrees
- moved C7 46.3 mm to (109.0, 96.0), turned to 270 degrees
- moved FID3 46.0 mm to (215.0, 51.0)
- moved JP1 43.6 mm to (124.0, 106.0), turned to 270 degrees
- moved C11 39.9 mm to (124.0, 95.0), turned to 270 degrees
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Connections:
- X1 pad 1: /ISOGND -> /ISOVCC
- X1 pad 2: /A -> /Z
- X1 pad 3: /B -> /Y
- X1 pad 4: /Y -> /B
- X1 pad 5: /Z -> /A
- X1 pad 6: /ISOVCC -> /ISOGND
Other:
- board outline added: 200 x 124 mm
- net class Default: clearance 0.8 -> 0.25
- rule trace_clearance: 0.8 -> 0.25
- board text added: "Fabricante MAYER: Ancho de pista: 0,8mm , 0,3mm Vias: 1,6mm/0,8mm Grillas: 1mm y 0.5mm posicionamiento 0.25mm ruteo Margen global: 0,8mm Terminacion: HASL"
- board text removed: "Fabricante MAYER: Ancho de pista: 0,8mm Vias: 1,6mm/0,8mm Margen global: 0,8mm"

Commit message: Version del PCB completa
Parts:
- added H1: MountingHole, MountingHole:MountingHole_2.1mm, F.Cu at (91.5, 80.0)
- added H2: MountingHole, MountingHole:MountingHole_2.1mm, F.Cu at (91.5, 106.0)
- added H3: MountingHole, MountingHole:MountingHole_2.1mm, F.Cu at (150.5, 80.0)
- added H4: MountingHole, MountingHole:MountingHole_2.1mm, F.Cu at (150.5, 106.0)
- C11, C3, C9: footprint Capacitor_Tantalum_SMD:CP_EIA-1608-08_AVX-J -> Capacitor_SMD:C_0805_2012Metric
- moved FID3 119.2 mm to (100.0, 82.5)
- moved FID1 111.6 mm to (99.8, 100.0)
- moved FID4 84.5 mm to (155.0, 102.5)
- moved FID2 60.1 mm to (155.0, 82.8)
- moved R1 40.2 mm to (142.2, 92.9), turned to 270 degrees
- moved R7 34.2 mm to (124.8, 97.2), turned to 180 degrees
- moved R2 32.5 mm to (150.1, 86.0), turned to 0 degrees
- moved R6 32.0 mm to (124.9, 87.8), turned to 180 degrees
- moved X1 31.3 mm to (162.8, 105.0)
- moved R5 30.6 mm to (124.9, 91.2), turned to 0 degrees
- moved R11 29.1 mm to (142.0, 98.2), turned to 270 degrees
- moved R3 29.1 mm to (124.9, 94.5)
- moved C2 29.1 mm to (137.2, 86.2)
- moved C5 29.1 mm to (133.3, 86.2)
- moved C1 27.9 mm to (129.3, 86.2)
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Connections:
- R1 pad 1: /B -> Net-(R1-Pad1)
- R1 pad 2: Net-(R1-Pad2) -> /B
- SW1 pad 1: Net-(R1-Pad2) -> /H_#F
- SW1 pad 2: /H_#F -> /A
- SW1 pad 5: /ISOGND -> Net-(R1-Pad1)
- SW1 pad 6: /A -> /ISOGND
- X1 pad 2: /Z -> /ISOGND
- X1 pad 3: /Y -> /Z
- X1 pad 4: /B -> /A
- X1 pad 5: /A -> /B
- X1 pad 6: /ISOGND -> /Y
- X2 pad 1: GND -> Net-(C9-Pad1)
- X2 pad 2: Net-(C9-Pad1) -> GND
Routing:
- net /ISOGND: track 0.00 -> 54.1 mm, vias 0 -> 2
- net /ISOVCC: track 0.00 -> 32.3 mm
- net /A: track 0.00 -> 31.3 mm
- net /B: track 0.00 -> 31.0 mm
- net /Y: track 0.00 -> 30.9 mm
- net VS: track 0.00 -> 29.7 mm, vias 0 -> 1
- net /Z: track 0.00 -> 27.8 mm
- net GND: track 0.00 -> 22.9 mm, vias 0 -> 4
- net Net-(C10-Pad2): track 0.00 -> 22.3 mm
- net +5V: track 0.00 -> 22.3 mm
- net /6_jmp: track 0.00 -> 19.5 mm, vias 0 -> 2
- net +3V3: track 0.00 -> 19.2 mm, vias 0 -> 1
- net /H_#F: track 0.00 -> 19.1 mm
- net /TX: track 0.00 -> 18.0 mm, vias 0 -> 1
- net /RX: track 0.00 -> 16.5 mm, vias 0 -> 1
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- added copper zone on B.Cu, net GND
- added copper zone on F.Cu, net GND
Other:
- board size 200 x 124 mm -> 77 x 31 mm
- board text added: "Fabricante MAYER: Ancho de pista: 0,3mm Vias: 1,6mm/0,8mm Grillas: 1mm y 0.5mm posicionamiento 0.25mm ruteo Margen global: 0,8mm Terminacion: HASL"
- board text removed: "Fabricante MAYER: Ancho de pista: 0,8mm , 0,3mm Vias: 1,6mm/0,8mm Grillas: 1mm y 0.5mm posicionamiento 0.25mm ruteo Margen global: 0,8mm Terminacion: HASL"

Commit message: Version para correccion
Other:
- board text added: "Creative Commons Attribution-ShareAlike 4.0 International License"
- board text added: "Fabricante MAYER: Ancho de pista: 0,3mm y 0,8mm Vias: 1,6mm/0,8mm Margen global: 0,25mm Terminacion: HASL Grillas: -1mm y 0.25mm posicionamiento -0.25mm ruteo"
- board text added: "[1 ]"
- board text added: "[2 ]"
- board text removed: "Fabricante MAYER: Ancho de pista: 0,3mm Vias: 1,6mm/0,8mm Grillas: 1mm y 0.5mm posicionamiento 0.25mm ruteo Margen global: 0,8mm Terminacion: HASL"
Changed lines of the file:
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@@
   (general
     (thickness 1.6)
-    (drawings 11)
+    (drawings 18)
     (tracks 206)
     (zones 0)
@@
   (page A4)
   (title_block
-    (title "Shield RS485")
+    (title "Shield RS485 para MKR1_Wifi1010")
     (date 11/4/21)
     (rev A)
@@
   )
   (setup
-    (last_trace_width 0.3)
+    (last_trace_width 0.8)
     (user_trace_width 0.3)
+    (user_trace_width 0.8)
     (trace_clearance 0.25)
     (zone_clearance 0.508)
@@
     (add_net VS)
   )
+  (module DO_214AC:DO-214BA (layer F.Cu)
+    (at 117.75 89.532 90)
+    (descr "<b>GF1</b><p>General Semiconductor")
+    (fp_text reference D1 (at 0.032 2.5 90) (layer F.SilkS)
+      (effects (font (size 1 1) (thickness 0.015)))
+    )
+    (fp_text value SS24FL (at -0.381 0 90) (layer F.Fab)
+      (effects (font (size 0.787402 0.787402) (thickness 0.015)))
+    )
+    (fp_line (start -2.9845 1.143) (end -2.9845 -1.143) (layer F.SilkS) (width 0.254))
+    (fp_line (start 2.9845 1.143) (end -2.9845 1.143) (layer F.SilkS) (width 0.254))
+    (fp_line (start 2.9845 -1.143) (end 2.9845 1.143) (layer F.SilkS) (width 0.254))
+    (fp_line (start -2.9845 -1.143) (end 2.9845 -1.143) (layer F.SilkS) (width 0.254))
+    (fp_line (start 0.635 0.762) (end 0.635 -0.762) (layer F.SilkS) (width 0.12))
+    (fp_line (start 0.635 -0.762) (end -0.635 0) (layer F.SilkS) (width 0.12))
+    (fp_line (start -0.635 0) (end 0.635 0.762) (layer F.SilkS) (width 0.12))
+    (fp_line (start -0.635 0.762) (end -0.635 -0.762) (layer F.SilkS) (width 0.12))
+    (pad 2 smd rect (at 2.0955 0 180) (size 1.8 1.34) (layers F.Cu F.Paste F.Mask)
+      (net 1 GND))
+    (pad 1 smd rect (at -2.0955 0 180) (size 1.8 1.34) (layers F.Cu F.Paste F.Mask)
+      (net 13 "Net-(C10-Pad2)"))
+    (model ${KIPRJMOD}/Librerias/DO_214AC/S1B.step
+      (offset (xyz 0 0 1.5))
+      (scale (xyz 1 1 1))
+      (rotate (xyz -90 0 0))
+    )
+  )
   (module MountingHole:MountingHole_2.1mm (layer F.Cu)
     (at 150.5 106)
@@
       (effects (font (size 1 1) (thickness 0.15)))
     )
-    (fp_text user %R (at 0.3 0) (layer F.Fab)
-      (effects (font (size 1 1) (thickness 0.15)))
-    )
     (fp_circle (center 0 0) (end 2.1 0) (layer Cmts.User) (width 0.15))
     (fp_circle (center 0 0) (end 2.35 0) (layer F.CrtYd) (width 0.05))
+    (fp_text user %R (at 0.3 0) (layer F.Fab)
+      (effects (font (size 1 1) (thickness 0.15)))
+    )
     (pad "" np_thru_hole circle (at 0 0) (size 2.1 2.1) (drill 2.1) (layers *.Cu *.Mask))
   )
@@
       (effects (font (size 1 1) (thickness 0.15)))
     )
-    (fp_text user %R (at 0.3 0) (layer F.Fab)
-      (effects (font (size 1 1) (thickness 0.15)))
-    )
     (fp_circle (center 0 0) (end 2.1 0) (layer Cmts.User) (width 0.15))
     (fp_circle (center 0 0) (end 2.35 0) (layer F.CrtYd) (width 0.05))
+    (fp_text user %R (at 0.3 0) (layer F.Fab)
+      (effects (font (size 1 1) (thickness 0.15)))
+    )
     (pad "" np_thru_hole circle (at 0 0) (size 2.1 2.1) (drill 2.1) (layers *.Cu *.Mask))
   )
@@
       (effects (font (size 1 1) (thickness 0.15)))
     )
-    (fp_text user %R (at 0.3 0) (layer F.Fab)
-      (effects (font (size 1 1) (thickness 0.15)))
-    )
     (fp_circle (center 0 0) (end 2.1 0) (layer Cmts.User) (width 0.15))
     (fp_circle (center 0 0) (end 2.35 0) (layer F.CrtYd) (width 0.05))
+    (fp_text user %R (at 0.3 0) (layer F.Fab)
+      (effects (font (size 1 1) (thickness 0.15)))
+    )
     (pad "" np_thru_hole circle (at 0 0) (size 2.1 2.1) (drill 2.1) (layers *.Cu *.Mask))
   )
@@
       (effects (font (size 1 1) (thickness 0.15)))
     )
-    (fp_text user %R (at 0.3 0) (layer F.Fab)
-      (effects (font (size 1 1) (thickness 0.15)))
-    )
     (fp_circle (center 0 0) (end 2.1 0) (layer Cmts.User) (width 0.15))
     (fp_circle (center 0 0) (end 2.35 0) (layer F.CrtYd) (width 0.05))
+    (fp_text user %R (at 0.3 0) (layer F.Fab)
+      (effects (font (size 1 1) (thickness 0.15)))
+    )
     (pad "" np_thru_hole circle (at 0 0) (size 2.1 2.1) (drill 2.1) (layers *.Cu *.Mask))
   )
@@
       (effects (font (size 1 1) (thickness 0.15)))
     )
-    (fp_text user %R (at 0 0 90) (layer F.Fab)
-      (effects (font (size 0.5 0.5) (thickness 0.08)))
-    )
     (fp_line (start -1 0.625) (end -1 -0.625) (layer F.Fab) (width 0.1))
     (fp_line (start -1 -0.625) (end 1 -0.625) (layer F.Fab) (width 0.1))
@@
     (fp_line (start 1.7 -0.98) (end 1.7 0.98) (layer F.CrtYd) (width 0.05))
     (fp_line (start 1.7 0.98) (end -1.7 0.98) (layer F.CrtYd) (width 0.05))
+    (fp_text user %R (at 0 0 90) (layer F.Fab)
+      (effects (font (size 0.5 0.5) (thickness 0.08)))
+    )
     (pad 2 smd roundrect (at 0.95 0 270) (size 1 1.45) (layers F.Cu F.Paste F.Mask) (roundrect_rratio 0.25)
       (net 1 GND))
@@
     (fp_text value 10u (at 0 1.68 90) (layer F.Fab)
       (effects (font (size 1 1) (thickness 0.15)))
-    )
-    (fp_text user %R (at 0 0 90) (layer F.Fab)
-      (effects (font (size 0.5 0.5) (thickness 0.08)))
     )
     (fp_line (start -1 0.625) (end -1 -0.625) (layer F.Fab) (width 0.1))
@@
     (fp_line (start 1.7 -0.98) (end 1.7 0.98) (layer F.CrtYd) (width 0.05))
     (fp_line (start 1.7 0.98) (end -1.7 0.98) (layer F.CrtYd) (width 0.05))
+    (fp_text user %R (at 0 0 90) (layer F.Fab)
+      (effects (font (size 0.5 0.5) (thickness 0.08)))
+    )
     (pad 2 smd roundrect (at 0.95 0 270) (size 1 1.45) (layers F.Cu F.Paste F.Mask) (roundrect_rratio 0.25)
       (net 1 GND))
@@
     (fp_text value 1u (at 0 1.68) (layer F.Fab)
       (effects (font (size 1 1) (thickness 0.15)))
-    )
-    (fp_text user %R (at 0 0) (layer F.Fab)
-      (effects (font (size 0.5 0.5) (thickness 0.08)))
     )
     (fp_line (start -1 0.625) (end -1 -0.625) (layer F.Fab) (width 0.1))
@@
     (fp_line (start 1.7 -0.98) (end 1.7 0.98) (layer F.CrtYd) (width 0.05))
     (fp_line (start 1.7 0.98) (end -1.7 0.98) (layer F.CrtYd) (width 0.05))
+    (fp_text user %R (at 0 0) (layer F.Fab)
+      (effects (font (size 0.5 0.5) (thickness 0.08)))
+    )
     (pad 2 smd roundrect (at 0.95 0) (size 1 1.45) (layers F.Cu F.Paste F.Mask) (roundrect_rratio 0.25)
       (net 3 /ISOGND))
@@
       (scale (xyz 1 1 1))
       (rotate (xyz 0 0 0))
-    )
-  )
-  (module DO_214AC:DO-214BA (layer F.Cu)
-    (at 117.75 89.532 90)
-    (descr "<b>GF1</b><p>General Semiconductor")
-    (fp_text reference D1 (at 0.032 2.5 90) (layer F.SilkS)
-      (effects (font (size 1 1) (thickness 0.015)))
-    )
-    (fp_text value SS24FL (at -0.381 0 90) (layer F.Fab)
-      (effects (font (size 0.787402 0.787402) (thickness 0.015)))
-    )
-    (fp_line (start -2.9845 -1.143) (end 2.9845 -1.143) (layer F.SilkS) (width 0.254))
-    (fp_line (start 2.9845 -1.143) (end 2.9845 1.143) (layer F.SilkS) (width 0.254))
-    (fp_line (start 2.9845 1.143) (end -2.9845 1.143) (layer F.SilkS) (width 0.254))
-    (fp_line (start -2.9845 1.143) (end -2.9845 -1.143) (layer F.SilkS) (width 0.254))
-    (pad 2 smd rect (at 2.0955 0 180) (size 1.8 1.34) (layers F.Cu F.Paste F.Mask)
-      (net 1 GND))
-    (pad 1 smd rect (at -2.0955 0 180) (size 1.8 1.34) (layers F.Cu F.Paste F.Mask)
-      (net 13 "Net-(C10-Pad2)"))
-    (model ${KIPRJMOD}/Librerias/DO_214AC/S1B.step
-      (offset (xyz 0 0 1.5))
-      (scale (xyz 1 1 1))
-      (rotate (xyz -90 0 0))
     )
   )
@@
     )
   )
+  (gr_text "[2 ]" (at 99.75 106.75) (layer B.Cu)
+    (effects (font (size 1.5 1.5) (thickness 0.3)) (justify mirror))
+  )
+  (gr_text "[1 ]" (at 99.75 106.75) (layer F.Cu)
+    (effects (font (size 1.5 1.5) (thickness 0.3)))
+  )
+  (gr_line (start 165.5 108.25) (end 165.25 77.75) (layer Margin) (width 0.15))
+  (gr_line (start 89 108.25) (end 165.5 108.25) (layer Margin) (width 0.15))
+  (gr_line (start 89 77.75) (end 89 108.25) (layer Margin) (width 0.15))
+  (gr_line (start 165.25 77.75) (end 89 77.75) (layer Margin) (width 0.15))
+  (gr_text "Creative Commons Attribution-ShareAlike 4.0 International License" (at 45.5 192.25) (layer Dwgs.User)
+    (effects (font (size 1 1) (thickness 0.15)))
+  )
   (gr_line (start 165.75 108.5) (end 165.75 108.25) (layer Edge.Cuts) (width 0.05))
   (gr_line (start 88.75 108.5) (end 165.75 108.5) (layer Edge.Cuts) (width 0.05))
@@
   (gr_line (start 88.75 77.5) (end 165.75 77.5) (layer Edge.Cuts) (width 0.05))
   (gr_line (start 88.75 108.25) (end 88.75 77.5) (layer Edge.Cuts) (width 0.05))
-  (gr_text "Fabricante MAYER:\nAncho de pista: 0,3mm\nVias: 1,6mm/0,8mm\n\nGrillas:\n1mm y 0.5mm posicionamiento\n0.25mm ruteo\nMargen global: 0,8mm\nTerminacion: HASL" (at 255 30) (layer Dwgs.User)
+  (gr_text "Fabricante MAYER:\nAncho de pista: 0,3mm y 0,8mm\nVias: 1,6mm/0,8mm\nMargen global: 0,25mm\nTerminacion: HASL\n\nGrillas:\n-1mm y 0.25mm posicionamiento\n-0.25mm ruteo\n" (at 255 30) (layer Dwgs.User)
     (effects (font (size 1 1) (thickness 0.15)) (justify left))
   )
@@
   (segment (start 98.21 88.365) (end 98 88.575) (width 0.3) (layer F.Cu) (net 12))
   (segment (start 101.525 88.365) (end 98.21 88.365) (width 0.3) (layer F.Cu) (net 12))
-  (segment (start 97.8375 88.5) (end 98 88.3375) (width 0.3) (layer F.Cu) (net 12))
-  (segment (start 91.25 88.5) (end 97.8375 88.5) (width 0.3) (layer F.Cu) (net 12))
+  (segment (start 97.8375 88.5) (end 98 88.3375) (width 0.8) (layer F.Cu) (net 12))
+  (segment (start 91.25 88.5) (end 97.8375 88.5) (width 0.8) (layer F.Cu) (net 12))
   (segment (start 98 85.2875) (end 102.7875 85.2875) (width 0.3) (layer F.Cu) (net 13))
   (segment (start 104.595 87.095) (end 106.475 87.095) (width 0.3) (layer F.Cu) (net 13))

Commit message: Version para corregir PCB
Parts:
- renumbered Interconexion1 to XA1
Connections:
- net /U2_FB renamed Net-(R10-Pad1)
Other:
- board text added: "Diseñado en Argentina"
