File: TP_DCI.kicad_pcb (KiCad board)
At the start: 2 copper layers, 77 x 31 mm, 42 parts, among them SW1 SW_DIP_x03, U1 MAX3157CAI+, U2 TPS54232, X1 Screw_Terminal_01x06, X2 Screw_Terminal_01x02

Commit message: Lista para correccion
Other:
- board text added: "Shield MKR1 v1"

Commit message: Agrego correcciones
Parts:
- removed FID3, FID4: Fiducial, Fiducial:Fiducial_0.5mm_Mask1.5mm
- moved H3 26.0 mm to (150.5, 106.0)
- moved H4 25.8 mm to (150.5, 80.2)
- moved R11 2.65 mm to (144.3, 99.5), turned to 180 degrees
- moved JP3 1.80 mm to (140.5, 85.5)
- moved JP4 1.77 mm to (146.5, 85.3)
- moved C3 1.25 mm to (138.6, 100.5)
- moved C1 1.25 mm to (129.3, 85.0)
- moved C2 1.25 mm to (137.2, 85.0)
- moved C4 1.25 mm to (134.8, 100.5)
- moved C5 1.25 mm to (133.3, 85.0)
- moved X1 0.74 mm to (162.8, 105.7)
- moved XA1 0.09 mm to (119.8, 92.8)
Routing:
- net /B: track 31.0 -> 37.3 mm, vias 0 -> 1
- net /ISOGND: track 54.1 -> 59.9 mm
- net /H_#F: track 19.1 -> 22.8 mm
- net /ISOVCC: track 32.3 -> 35.7 mm, vias 0 -> 1
- net /6_jmp: track 19.5 -> 22.1 mm
- net /Y: track 30.9 -> 28.6 mm
- net GND: track 22.9 -> 25.1 mm, vias 4 -> 5
- net /A: track 31.3 -> 33.2 mm
- net /7: track 1.96 -> 3.54 mm
- net /6: track 1.96 -> 3.46 mm
- net +5V: track 22.3 -> 23.6 mm
- net Net-(C5-Pad2): track 3.55 -> 4.80 mm
- net Net-(C5-Pad1): track 3.53 -> 4.78 mm
- net Net-(C4-Pad2): track 3.17 -> 4.42 mm
- net Net-(C4-Pad1): track 3.19 -> 4.44 mm
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Other:
- net class Default: clearance 0.25 -> 0.35
- rule trace_clearance: 0.25 -> 0.35
- board text added: "Fabricante MAYER: Ancho de pista: 0,3mm y 0,8mm Vias: 0,8mm/0,4mm Margen global: 0,25mm Terminacion: HASL Grillas: -1mm y 0.25mm posicionamiento -0.25mm ruteo"
- board text removed: "Fabricante MAYER: Ancho de pista: 0,3mm y 0,8mm Vias: 1,6mm/0,8mm Margen global: 0,25mm Terminacion: HASL Grillas: -1mm y 0.25mm posicionamiento -0.25mm ruteo"

Commit message: Agrego correcciones finales
Parts:
- X2: footprint TerminalBlock_Phoenix:TerminalBlock_Phoenix_MKDS-1,5-2-5.08_1x02_P5.08mm_Horizontal -> TerminalBlock:TerminalBlock_bornier-2_P5.08mm
